File: discodolly.brd (EAGLE design)
At the start: 150 x 100 mm, 25 parts, among them T1 BC337

Commit message: approve overlaps
Routing:
- net WS2812: track 6.00 -> 7.25 mm
- net VCC: track 68.9 -> 70.1 mm
Changed lines of the file:
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@@
 <?xml version="1.0" encoding="utf-8"?>
 <!DOCTYPE eagle SYSTEM "eagle.dtd">
-<eagle version="9.3.2">
+<eagle version="9.4.0">
 <drawing>
 <settings>
@@
 <layer number="14" name="Route14" color="22" fill="1" visible="no" active="no"/>
 <layer number="15" name="Route15" color="23" fill="1" visible="no" active="no"/>
-<layer number="16" name="Bottom" color="1" fill="1" visible="yes" active="yes"/>
+<layer number="16" name="Bottom" color="1" fill="1" visible="no" active="yes"/>
 <layer number="17" name="Pads" color="2" fill="1" visible="yes" active="yes"/>
-<layer number="18" name="Vias" color="2" fill="1" visible="yes" active="yes"/>
+<layer number="18" name="Vias" color="2" fill="1" visible="no" active="yes"/>
 <layer number="19" name="Unrouted" color="6" fill="1" visible="yes" active="yes"/>
 <layer number="20" name="Dimension" color="24" fill="1" visible="yes" active="yes"/>
-<layer number="21" name="tPlace" color="7" fill="1" visible="yes" active="yes"/>
-<layer number="22" name="bPlace" color="7" fill="1" visible="yes" active="yes"/>
-<layer number="23" name="tOrigins" color="15" fill="1" visible="yes" active="yes"/>
-<layer number="24" name="bOrigins" color="15" fill="1" visible="yes" active="yes"/>
-<layer number="25" name="tNames" color="7" fill="1" visible="yes" active="yes"/>
-<layer number="26" name="bNames" color="7" fill="1" visible="yes" active="yes"/>
+<layer number="21" name="tPlace" color="7" fill="1" visible="no" active="yes"/>
+<layer number="22" name="bPlace" color="7" fill="1" visible="no" active="yes"/>
+<layer number="23" name="tOrigins" color="15" fill="1" visible="no" active="yes"/>
+<layer number="24" name="bOrigins" color="15" fill="1" visible="no" active="yes"/>
+<layer number="25" name="tNames" color="7" fill="1" visible="no" active="yes"/>
+<layer number="26" name="bNames" color="7" fill="1" visible="no" active="yes"/>
 <layer number="27" name="tValues" color="7" fill="1" visible="no" active="yes"/>
 <layer number="28" name="bValues" color="7" fill="1" visible="no" active="yes"/>
@@
 <layer number="37" name="tTest" color="7" fill="1" visible="no" active="yes"/>
 <layer number="38" name="bTest" color="7" fill="1" visible="no" active="yes"/>
-<layer number="39" name="tKeepout" color="4" fill="11" visible="yes" active="yes"/>
-<layer number="40" name="bKeepout" color="1" fill="11" visible="yes" active="yes"/>
-<layer number="41" name="tRestrict" color="4" fill="10" visible="yes" active="yes"/>
-<layer number="42" name="bRestrict" color="1" fill="10" visible="yes" active="yes"/>
+<layer number="39" name="tKeepout" color="4" fill="11" visible="no" active="yes"/>
+<layer number="40" name="bKeepout" color="1" fill="11" visible="no" active="yes"/>
+<layer number="41" name="tRestrict" color="4" fill="10" visible="no" active="yes"/>
+<layer number="42" name="bRestrict" color="1" fill="10" visible="no" active="yes"/>
 <layer number="43" name="vRestrict" color="2" fill="10" visible="no" active="yes"/>
 <layer number="44" name="Drills" color="7" fill="1" visible="no" active="yes"/>
-<layer number="45" name="Holes" color="7" fill="1" visible="yes" active="yes"/>
+<layer number="45" name="Holes" color="7" fill="1" visible="no" active="yes"/>
 <layer number="46" name="Milling" color="3" fill="1" visible="no" active="yes"/>
 <layer number="47" name="Measures" color="7" fill="1" visible="no" active="yes"/>
@@
 <layer number="49" name="Reference" color="7" fill="1" visible="no" active="yes"/>
 <layer number="50" name="dxf" color="7" fill="1" visible="no" active="yes"/>
-<layer number="51" name="tDocu" color="7" fill="1" visible="yes" active="yes"/>
-<layer number="52" name="bDocu" color="7" fill="1" visible="yes" active="yes"/>
+<layer number="51" name="tDocu" color="7" fill="1" visible="no" active="yes"/>
+<layer number="52" name="bDocu" color="7" fill="1" visible="no" active="yes"/>
 <layer number="53" name="tGND_GNDA" color="7" fill="9" visible="no" active="no"/>
 <layer number="54" name="bGND_GNDA" color="1" fill="9" visible="no" active="no"/>
@@
 <contactref element="TP4" pad="TP"/>
 <wire x1="3.5" y1="66.15" x2="-2.4" y2="66.15" width="1.27" layer="1"/>
-<wire x1="-2.4" y1="66.15" x2="-3.75" y2="65" width="1.27" layer="1"/>
-<wire x1="-2.4" y1="66.15" x2="-2.5" y2="65" width="0" layer="19" extent="1-1"/>
+<wire x1="-3.75" y1="65" x2="-2.4" y2="66.15" width="1.27" layer="1"/>
+<wire x1="-2.4" y1="66.15" x2="-2.4" y2="65" width="0.1524" layer="1"/>
+<wire x1="-2.4" y1="65" x2="-2.5" y2="65" width="0.1524" layer="1"/>
 </signal>
 <signal name="N$2">
@@
 <contactref element="TP2" pad="TP"/>
 <contactref element="SV2" pad="4"/>
-<wire x1="-3.75" y1="71.25" x2="-2.5" y2="71.25" width="0" layer="19" extent="1-1"/>
+<wire x1="-3.75" y1="71.25" x2="-2.5" y2="71.25" width="0.1524" layer="1"/>
 </signal>
 <signal name="MODE">
@@
 <wire x1="3.5" y1="76.31" x2="-7.44" y2="76.31" width="1.27" layer="1"/>
 <wire x1="-7.44" y1="76.31" x2="-7.5" y2="76.25" width="1.27" layer="1"/>
-<wire x1="-7.7394" y1="78.2512" x2="-7.7394" y2="71.7488" width="1.27" layer="1"/>
-<wire x1="-7.7394" y1="78.2512" x2="-7.44" y2="76.31" width="0" layer="19" extent="1-1"/>
+<wire x1="-7.7394" y1="71.7488" x2="-7.7394" y2="76.25" width="1.27" layer="1"/>
+<wire x1="-7.7394" y1="76.25" x2="-7.7394" y2="78.2512" width="1.27" layer="1"/>
+<wire x1="-7.7394" y1="76.25" x2="-7.6794" y2="76.31" width="1.27" layer="1"/>
+<wire x1="-7.6794" y1="76.31" x2="-7.44" y2="76.31" width="1.27" layer="1"/>
+</signal>
+<signal name="N$6">
+<via x="-10" y="75" extent="1-16" drill="0.35"/>
 </signal>
 </signals>
@@
 <mfgpreviewcolor name="substratecolor" color="0xFF786E46"/>
 </mfgpreviewcolors>
+<errors>
+</errors>
 </board>
 </drawing>
